File: pcb/flashlight.kicad_pcb (KiCad board)
At the start: 2 copper layers, 16.8 x 15.8 mm, 25 parts, among them IC1 TPS61200, IC2 PIC10F320

Commit message: replace 10k with 470k
Parts:
- R2: value 10k -> 470k
Changed lines of the file:
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@@
       (effects (font (size 0.8 0.8) (thickness 0.16)))
     )
-    (fp_text value 10k (at -1.2 0 270) (layer F.Fab)
+    (fp_text value 470k (at -1.2 0 270) (layer F.Fab)
       (effects (font (size 0.6 0.6) (thickness 0.12)))
     )

Commit message: connect R2 to GND
Parts:
- R2: value 470k -> 1M
Connections:
- R2 pad 1: N$4 -> GND
Routing:
- net N$4: track 12.7 -> 10.6 mm
- net GND: track 7.04 -> 8.79 mm
Changed lines of the file:
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@@
   (general
     (links 38)
-    (no_connects 23)
+    (no_connects 24)
     (area 141.528103 92.033521 158.471897 107.966479)
     (thickness 1.6)
     (drawings 11)
-    (tracks 77)
+    (tracks 75)
     (zones 0)
     (modules 25)
@@
   )
   (setup
-    (last_trace_width 0.25)
+    (last_trace_width 1)
     (user_trace_width 0.5)
     (user_trace_width 1)
@@
     (pad_to_mask_clearance 0.2)
     (aux_axis_origin 0 0)
-    (visible_elements 7FFFFFFF)
+    (visible_elements 7FFCFFFF)
     (pcbplotparams
       (layerselection 0x01030_80000001)
@@
       (effects (font (size 0.8 0.8) (thickness 0.16)))
     )
-    (fp_text value 470k (at -1.2 0 270) (layer F.Fab)
+    (fp_text value 1M (at -1.2 0 270) (layer F.Fab)
       (effects (font (size 0.6 0.6) (thickness 0.12)))
     )
     (pad 1 smd rect (at -1 0 270) (size 1 1.3) (layers F.Cu F.Paste F.Mask)
-      (net 6 N$4))
+      (net 2 GND))
     (pad 2 smd rect (at 1 0 270) (size 1 1.3) (layers F.Cu F.Paste F.Mask)
       (net 3 N$3))
@@
   (segment (start 153 103.9) (end 153 102.6) (width 0.25) (layer F.Cu) (net 1))
   (segment (start 152.6 104.3) (end 153 103.9) (width 0.25) (layer F.Cu) (net 1))
+  (segment (start 154.75 99) (end 156.5 99) (width 0.25) (layer F.Cu) (net 2))
   (segment (start 149.05 104.8) (end 150.25 104.8) (width 0.25) (layer F.Cu) (net 2))
   (segment (start 150.25 104.8) (end 150.5 104.55) (width 0.25) (layer F.Cu) (net 2))
@@
   (via (at 154.56 102.6) (size 0.6) (drill 0.4) (layers F.Cu B.Cu) (net 3))
   (segment (start 147.2 96.9) (end 145 96.9) (width 1.5) (layer F.Cu) (net 5))
-  (segment (start 153.7 101.55) (end 153.7 100.05) (width 0.25) (layer F.Cu) (net 6))
   (segment (start 153.3 101.95) (end 153.7 101.55) (width 0.25) (layer F.Cu) (net 6))
+  (segment (start 153.3 100.05) (end 152.475 100.05) (width 0.25) (layer F.Cu) (net 6))
+  (segment (start 153.7 100.45) (end 153.3 100.05) (width 0.25) (layer F.Cu) (net 6))
+  (segment (start 153.7 101.55) (end 153.7 100.45) (width 0.25) (layer F.Cu) (net 6))
   (segment (start 153.7 102.35) (end 153.7 103.72) (width 0.25) (layer F.Cu) (net 6))
   (segment (start 151.27 105.09) (end 152.16 104.79) (width 0.25) (layer B.Cu) (net 6))
@@
   (segment (start 153.25 101.95) (end 153.3 101.95) (width 0.25) (layer F.Cu) (net 6))
   (segment (start 153.3 101.95) (end 153.7 102.35) (width 0.25) (layer F.Cu) (net 6))
-  (segment (start 154.75 99) (end 154.75 99.75) (width 0.25) (layer F.Cu) (net 6))
-  (segment (start 154.75 99.75) (end 154.45 100.05) (width 0.25) (layer F.Cu) (net 6))
-  (segment (start 154.45 100.05) (end 153.7 100.05) (width 0.25) (layer F.Cu) (net 6))
-  (segment (start 153.7 100.05) (end 153.5 100.05) (width 0.25) (layer F.Cu) (net 6))
-  (segment (start 153.5 100.05) (end 152.475 100.05) (width 0.25) (layer F.Cu) (net 6))
   (segment (start 151.95 103.8) (end 151.95 103.5) (width 0.25) (layer F.Cu) (net 6))
   (segment (start 151.95 103.5) (end 152.3 103.15) (width 0.25) (layer F.Cu) (net 6))
